Commit message: add maps to velmwheel_description, add laser_configuration xacro

File: velmwheel_description/urdf/velmobil_laser_poses.xacro (robot description, xacro)
@@ -2,5 +2,5 @@
 <robot xmlns:xacro="http://www.ros.org/wiki/xacro" name="velmobil">
 <xacro:property name="front_laser_origin_from_calibration">
-   <origin xyz="0 0 0" rpy="0 0 0" />
+   <origin xyz="0.3 -0.0113536 0" rpy="0 0 0" />
 </xacro:property>
 <xacro:property name="rear_laser_origin_from_calibration">
