Commit message: add velmobil mesh

File: velmwheel_description/urdf/velmobil.urdf.xacro (robot description, xacro)
@@ -3,5 +3,11 @@
 <!-- INCLUDE LMX100 LASER CALIBRATION DATA-->
 <xacro:include filename="$(find velmwheel_description)/urdf/velmobil_laser_poses.xacro" />
-  <link name="base_link" />
+  <link name="base_link">
+     	<visual>
+	  <geometry>
+	    <mesh filename="package://velmwheel_description/meshes/velmobil_scaled.dae"/>
+	  </geometry>
+	</visual>
+  </link>
   <link name="odom" />
   <link name="laser_front_link" />

Commit message: new mesh, new amcl params, add mesh to xacro

File: velmwheel_description/urdf/velmobil.urdf.xacro (robot description, xacro)
@@ -6,5 +6,5 @@
      	<visual>
 	  <geometry>
-	    <mesh filename="package://velmwheel_description/meshes/velmobil_scaled.dae"/>
+	    <mesh filename="package://velmwheel_description/meshes/velmobil_scaled_2.stl"/>
 	  </geometry>
 	</visual>
